File: SmartChessboard_Hardware/SmartChessboard.kicad_sch (KiCad schematic)
At the start: 0 parts

Commit message: first test
Other:
- title: (none) -> SmartChessboard
Changed lines of the file:
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@@
 	(generator_version "9.0")
 	(paper "A4")
+	(title_block
+		(title "SmartChessboard")
+		(date "2025-08-24")
+		(rev "0")
+		(comment 1 "Releases under CERN Open Hardware Licence Version 2")
+	)
 	(sheet_instances
 		(path "/"
