File: SmartChessboard_PCB/peripherals.kicad_sch (KiCad schematic)
At the start: 22 parts, among them J2 Qwiic_RA, J3 JST_2mm_LiPo, U4 RT9080-3.3, U5 MCP73831, U6 MAX17048

Commit message: before hall sensors
Parts:
- removed C9: 0.1uF, SparkFun-Capacitor:C_0402_1005Metric, symbol SparkFun-Capacitor:0.1uF_0402_6.3V_10%
- removed D5: WS2812B, SparkFun-LED:WS2812_2020, symbol SparkFun-LED:WS2812B_2020
- removed TP2: 1.0mm, SparkFun-Connector:TestPoint-1.0mm, symbol SparkFun-Connector:TestPoint_1.0mm
Other:
- note removed: "RGB LED"

Commit message: level shifter added
Other:
- title: (none) -> SmartChessboard
Changed lines of the file:
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@@
 	(generator_version "9.0")
 	(paper "A4")
+	(title_block
+		(title "SmartChessboard")
+		(date "2025-08-15")
+		(rev "0")
+		(comment 3 "Released under CERN Open Hardware Licence Version 2")
+		(comment 4 "Designed by: Alessandro Sabbadini")
+	)
 	(text "Charge current:\nI_CHG = 1000 / R_PROG\nR_PROG=2k : I_CHG=500mA"
 		(exclude_from_sim no)

Commit message: psc
Parts:
- removed C10: 4.7uF, SparkFun-Capacitor:C_0603_1608Metric, symbol SparkFun-Capacitor:4.7uF_0603_35V_20%
- removed C11: 0.1uF, SparkFun-Capacitor:C_0402_1005Metric, symbol SparkFun-Capacitor:0.1uF_0402_6.3V_10%
- removed C12: 4.7uF, SparkFun-Capacitor:C_0402_1005Metric, symbol SparkFun-Capacitor:4.7uF_0402_6.3V_10%
- removed D6: Yellow, SparkFun-LED:LED_0603_1608Metric_Yellow, symbol SparkFun-LED:LED_Yellow_0603
- removed J2: Qwiic_RA, SparkFun-Connector:JST_SMD_1.0mm-4_RA, symbol SparkFun-Connector:Qwiic_Right_Angle
- removed J3: JST_2mm_LiPo, SparkFun-Connector:JST_SMD_2.0mm-2, symbol SparkFun-Connector:Conn_01x02_JST_2mm_LiPo
- removed JP3: ~, SparkFun-Jumper:Jumper_2_NC_Trace, symbol SparkFun-Jumper:SolderJumper_2_Bridged
- removed R11: 1k, SparkFun-Resistor:R_0402_1005Metric, symbol SparkFun-Resistor:1k_0402
- removed R12: 2.0k, SparkFun-Resistor:R_0402_1005Metric, symbol SparkFun-Resistor:2.0k_0402
- removed U5: MCP73831, SparkFun-Semiconductor-Standard:SOT23-5, symbol SparkFun-IC-Power:MCP73831
- removed U6: MAX17048, SparkFun-Semiconductor-Standard:DFN-8, symbol SparkFun-IC-Power:MAX17048
- added J4, J6: I2C, SparkFun-Connector:1x04, symbol SparkFun-Connector:I2C_01x04
- added J5: FRJAE438, FRJAE438:AMPHENOL_FRJAE438, symbol FRJAE438:FRJAE438
Connections:
- net 3.3V_P: now also J4.2 (Pin_2)
- net ESP8/SDA: now also J4.3 (Pin_3)
- net ESP9/SCL: now also J4.4 (Pin_4)
- net GND: now also J4.1 (Pin_1), J5.4
- new net: J5.5, J6.1 (Pin_1)
- new net: J5.6, J6.2 (Pin_2)
- new net: J5.7, J6.3 (Pin_3)
- new net: J5.8, J6.4 (Pin_4)
- new net: J5.SH1 (SHIELD), J5.SH2 (SHIELD)
- new net ESP43/TXO: J5.3
- new net ESP44/RXI: J5.2
- new net VDOBOT: J5.1
- no-connect marks 0 -> 1
Other:
- note removed: "7-bit I2C Address: 0x36"
- note removed: "Charge current: I_CHG = 1000 / R_PROG R_PROG=2k : I_CHG=500mA"
- note removed: "Fuel Gauge"
- note removed: "LiPo Charger"
