File: SmartChessboard_PCB/hall.kicad_sch (KiCad schematic)
At the start: 0 parts

Commit message: level shifter added
Parts:
- added C100, C101, C110, C111, C112, C113, C114, C115, C116, C117, C126, C127, C128, C129, C130, C131, C132, C140, C141, C142, C143, C144, C145, C146, C147, C156, C157, C158, C159, C160, C161, C162, C163, C172, C173, C174, C175, C176, C177, C178, C179, C188, C189, C190, C191, C192, C193, C194, C195, C78, C79, C80, C81, C82, C83, C84, C85, C9, C94, C95, C96, C97, C98, C99: 100nF, PCM_JLCPCB:C_0402, symbol PCM_JLCPCB-Capacitors:0402,100nF,(2)
- added C102, C103, C104, C105, C106, C107, C108, C109, C118, C119, C120, C121, C122, C123, C124, C125, C13, C133, C134, C135, C136, C137, C138, C139, C148, C149, C150, C151, C152, C153, C154, C155, C164, C165, C166, C167, C168, C169, C170, C171, C180, C181, C182, C183, C184, C185, C186, C187, C196, C197, C198, C199, C200, C201, C202, C203, C86, C87, C88, C89, C90, C91, C92, C93: 4.7nF, PCM_JLCPCB:C_0402, symbol PCM_JLCPCB-Capacitors:0402,4.7nF
- added R13, R14, R15, R16, R17, R18, R19, R20, R21, R22, R23, R24, R25, R26, R27, R28, R29, R30, R31, R32, R33, R34, R35, R36, R37, R38, R39, R40, R41, R42, R43, R44, R45, R46, R47, R48, R49, R50, R51, R52, R53, R54, R55, R56, R57, R58, R59, R60, R61, R62, R63, R64, R65, R66, R67, R68, R69, R70, R71, R72, R73, R74, R75, R76: 10k, SparkFun-Resistor:R_0402_1005Metric, symbol SparkFun-Resistor:10k_0402
- added U10, U11, U7, U8: CD74HC4067, SparkFun-Semiconductor-Standard:TSSOP-24_4.4x7.8mm_P0.65mm, symbol SparkFun-IC-Special-Function:CD74HC4067
- added U12: TXB0104D, Package_SO:SOIC-14_3.9x8.7mm_P1.27mm, symbol Logic_LevelTranslator:TXB0104D
- added U14, U15, U16, U17, U18, U19, U20, U21, U22, U23, U24, U25, U26, U27, U28, U29, U30, U31, U32, U33, U34, U35, U36, U37, U38, U39, U40, U41, U42, U43, U44, U45, U46, U47, U48, U49, U50, U51, U52, U53, U54, U55, U56, U57, U58, U59, U60, U61, U62, U63, U64, U65, U66, U67, U68, U69, U70, U71, U72, U73, U74, U75, U76, U9: US5881ESE-AAA-000-RE, US5881ESE-AAA-000-RE:SOT95P280X100-3N, symbol US5881ESE-AAA-000-RE:US5881ESE-AAA-000-RE
Connections:
- new net 3.3V: U12.1 (VCCA)
- new net 5V: C100.1, C101.1, C110.1, C111.1, C112.1, C113.1, C114.1, C115.1, C116.1, C117.1, C126.1, C127.1, C128.1, C129.1, C130.1, C131.1, C132.1, C140.1, C141.1, C142.1, C143.1, C144.1, C145.1, C146.1, C147.1, C156.1, C157.1, C158.1, C159.1, C160.1, C161.1, C162.1, C163.1, C172.1, C173.1, C174.1, C175.1, C176.1, C177.1, C178.1, C179.1, C188.1, C189.1, C190.1, C191.1, C192.1, C193.1, C194.1, C195.1, C78.1, C79.1, C80.1, C81.1, C82.1, C83.1, C84.1, C85.1, C9.1, C94.1, C95.1, C96.1, C97.1, C98.1, C99.1, R13.2, R14.2, R15.2, R16.2, R17.2, R18.2, R19.2, R20.2, R21.2, R22.2, R23.2, R24.2, R25.2, R26.2, R27.2, R28.2, R29.2, R30.2, R31.2, R32.2, R33.2, R34.2, R35.2, R36.2, R37.2, R38.2, R39.2, R40.2, R41.2, R42.2, R43.2, R44.2, R45.2, R46.2, R47.2, R48.2, R49.2, R50.2, R51.2, R52.2, R53.2, R54.2, R55.2, R56.2, R57.2, R58.2, R59.2, R60.2, R61.2, R62.2, R63.2, R64.2, R65.2, R66.2, R67.2, R68.2, R69.2, R70.2, R71.2, R72.2, R73.2, R74.2, R75.2, R76.2, U10.24 (VCC), U11.24 (VCC), U12.14 (VCCB), U14.1 (VDD), U15.1 (VDD), U16.1 (VDD), U17.1 (VDD), U18.1 (VDD), U19.1 (VDD), U20.1 (VDD), U21.1 (VDD), U22.1 (VDD), U23.1 (VDD), U24.1 (VDD), U25.1 (VDD), U26.1 (VDD), U27.1 (VDD), U28.1 (VDD), U29.1 (VDD), U30.1 (VDD), U31.1 (VDD), U32.1 (VDD), U33.1 (VDD), U34.1 (VDD), U35.1 (VDD), U36.1 (VDD), U37.1 (VDD), U38.1 (VDD), U39.1 (VDD), U40.1 (VDD), U41.1 (VDD), U42.1 (VDD), U43.1 (VDD), U44.1 (VDD), U45.1 (VDD), U46.1 (VDD), U47.1 (VDD), U48.1 (VDD), U49.1 (VDD), U50.1 (VDD), U51.1 (VDD), U52.1 (VDD), U53.1 (VDD), U54.1 (VDD), U55.1 (VDD), U56.1 (VDD), U57.1 (VDD), U58.1 (VDD), U59.1 (VDD), U60.1 (VDD), U61.1 (VDD), U62.1 (VDD), U63.1 (VDD), U64.1 (VDD), U65.1 (VDD), U66.1 (VDD), U67.1 (VDD), U68.1 (VDD), U69.1 (VDD), U7.24 (VCC), U70.1 (VDD), U71.1 (VDD), U72.1 (VDD), U73.1 (VDD), U74.1 (VDD), U75.1 (VDD), U76.1 (VDD), U8.24 (VCC), U9.1 (VDD)
- new net GND: C100.2, C101.2, C102.2, C103.2, C104.2, C105.2, C106.2, C107.2, C108.2, C109.2, C110.2, C111.2, C112.2, C113.2, C114.2, C115.2, C116.2, C117.2, C118.2, C119.2, C120.2, C121.2, C122.2, C123.2, C124.2, C125.2, C126.2, C127.2, C128.2, C129.2, C13.2, C130.2, C131.2, C132.2, C133.2, C134.2, C135.2, C136.2, C137.2, C138.2, C139.2, C140.2, C141.2, C142.2, C143.2, C144.2, C145.2, C146.2, C147.2, C148.2, C149.2, C150.2, C151.2, C152.2, C153.2, C154.2, C155.2, C156.2, C157.2, C158.2, C159.2, C160.2, C161.2, C162.2, C163.2, C164.2, C165.2, C166.2, C167.2, C168.2, C169.2, C170.2, C171.2, C172.2, C173.2, C174.2, C175.2, C176.2, C177.2, C178.2, C179.2, C180.2, C181.2, C182.2, C183.2, C184.2, C185.2, C186.2, C187.2, C188.2, C189.2, C190.2, C191.2, C192.2, C193.2, C194.2, C195.2, C196.2, C197.2, C198.2, C199.2, C200.2, C201.2, C202.2, C203.2, C78.2, C79.2, C80.2, C81.2, C82.2, C83.2, C84.2, C85.2, C86.2, C87.2, C88.2, C89.2, C9.2, C90.2, C91.2, C92.2, C93.2, C94.2, C95.2, C96.2, C97.2, C98.2, C99.2, U10.12 (GND), U10.15 (~{EN}), U11.12 (GND), U11.15 (~{EN}), U12.7 (GND), U14.3 (GND), U15.3 (GND), U16.3 (GND), U17.3 (GND), U18.3 (GND), U19.3 (GND), U20.3 (GND), U21.3 (GND), U22.3 (GND), U23.3 (GND), U24.3 (GND), U25.3 (GND), U26.3 (GND), U27.3 (GND), U28.3 (GND), U29.3 (GND), U30.3 (GND), U31.3 (GND), U32.3 (GND), U33.3 (GND), U34.3 (GND), U35.3 (GND), U36.3 (GND), U37.3 (GND), U38.3 (GND), U39.3 (GND), U40.3 (GND), U41.3 (GND), U42.3 (GND), U43.3 (GND), U44.3 (GND), U45.3 (GND), U46.3 (GND), U47.3 (GND), U48.3 (GND), U49.3 (GND), U50.3 (GND), U51.3 (GND), U52.3 (GND), U53.3 (GND), U54.3 (GND), U55.3 (GND), U56.3 (GND), U57.3 (GND), U58.3 (GND), U59.3 (GND), U60.3 (GND), U61.3 (GND), U62.3 (GND), U63.3 (GND), U64.3 (GND), U65.3 (GND), U66.3 (GND), U67.3 (GND), U68.3 (GND), U69.3 (GND), U7.12 (GND), U7.15 (~{EN}), U70.3 (GND), U71.3 (GND), U72.3 (GND), U73.3 (GND), U74.3 (GND), U75.3 (GND), U76.3 (GND), U8.12 (GND), U8.15 (~{EN}), U9.3 (GND)
- new net Hall_1: C102.1, C103.1, C104.1, C105.1, C106.1, C107.1, C108.1, C109.1, C118.1, C119.1, C120.1, C121.1, C122.1, C123.1, C124.1, C125.1, C13.1, C133.1, C134.1, C135.1, C136.1, C137.1, C138.1, C139.1, C148.1, C149.1, C150.1, C151.1, C152.1, C153.1, C154.1, C155.1, C164.1, C165.1, C166.1, C167.1, C168.1, C169.1, C170.1, C171.1, C180.1, C181.1, C182.1, C183.1, C184.1, C185.1, C186.1, C187.1, C196.1, C197.1, C198.1, C199.1, C200.1, C201.1, C202.1, C203.1, C86.1, C87.1, C88.1, C89.1, C90.1, C91.1, C92.1, C93.1, R13.1, R14.1, R15.1, R16.1, R17.1, R18.1, R19.1, R20.1, R21.1, R22.1, R23.1, R24.1, R25.1, R26.1, R27.1, R28.1, R29.1, R30.1, R31.1, R32.1, R33.1, R34.1, R35.1, R36.1, R37.1, R38.1, R39.1, R40.1, R41.1, R42.1, R43.1, R44.1, R45.1, R46.1, R47.1, R48.1, R49.1, R50.1, R51.1, R52.1, R53.1, R54.1, R55.1, R56.1, R57.1, R58.1, R59.1, R60.1, R61.1, R62.1, R63.1, R64.1, R65.1, R66.1, R67.1, R68.1, R69.1, R70.1, R71.1, R72.1, R73.1, R74.1, R75.1, R76.1, U14.2 (OUT), U7.9 (I0)
- new net Hall_10: U23.2 (OUT), U7.22 (I9)
- new net Hall_11: U31.2 (OUT), U7.21 (I10)
- new net Hall_12: U38.2 (OUT), U7.20 (I11)
- new net Hall_13: U46.2 (OUT), U7.19 (I12)
- new net Hall_14: U54.2 (OUT), U7.18 (I13)
- new net Hall_15: U62.2 (OUT), U7.17 (I14)
- new net Hall_16: U7.16 (I15), U70.2 (OUT)
- new net Hall_17: U16.2 (OUT), U8.9 (I0)
- new net Hall_18: U24.2 (OUT), U8.8 (I1)
- new net Hall_19: U32.2 (OUT), U8.7 (I2)
- new net Hall_2: U22.2 (OUT), U7.8 (I1)
- new net Hall_20: U39.2 (OUT), U8.6 (I3)
- new net Hall_21: U47.2 (OUT), U8.5 (I4)
- new net Hall_22: U55.2 (OUT), U8.4 (I5)
- new net Hall_23: U63.2 (OUT), U8.3 (I6)
- new net Hall_24: U71.2 (OUT), U8.2 (I7)
- new net Hall_25: U17.2 (OUT), U8.23 (I8)
- new net Hall_26: U25.2 (OUT), U8.22 (I9)
- new net Hall_27: U33.2 (OUT), U8.21 (I10)
- new net Hall_28: U40.2 (OUT), U8.20 (I11)
- new net Hall_29: U48.2 (OUT), U8.19 (I12)
- new net Hall_3: U30.2 (OUT), U7.7 (I2)
- new net Hall_30: U56.2 (OUT), U8.18 (I13)
- new net Hall_31: U64.2 (OUT), U8.17 (I14)
- new net Hall_32: U72.2 (OUT), U8.16 (I15)
- new net Hall_33: U10.9 (I0), U18.2 (OUT)
- new net Hall_34: U10.8 (I1), U26.2 (OUT)
- new net Hall_35: U10.7 (I2), U34.2 (OUT)
- new net Hall_36: U10.6 (I3), U41.2 (OUT)
- new net Hall_37: U10.5 (I4), U49.2 (OUT)
- new net Hall_38: U10.4 (I5), U57.2 (OUT)
- new net Hall_39: U10.3 (I6), U65.2 (OUT)
- new net Hall_4: U7.6 (I3), U9.2 (OUT)
- new net Hall_40: U10.2 (I7), U73.2 (OUT)
- new net Hall_41: U10.23 (I8), U19.2 (OUT)
- new net Hall_42: U10.22 (I9), U27.2 (OUT)
- new net Hall_43: U10.21 (I10), U35.2 (OUT)
- new net Hall_44: U10.20 (I11), U42.2 (OUT)
- new net Hall_45: U10.19 (I12), U50.2 (OUT)
- new net Hall_46: U10.18 (I13), U58.2 (OUT)
- new net Hall_47: U10.17 (I14), U66.2 (OUT)
- new net Hall_48: U10.16 (I15), U74.2 (OUT)
- new net Hall_49: U11.9 (I0), U20.2 (OUT)
- new net Hall_5: U45.2 (OUT), U7.5 (I4)
- new net Hall_50: U11.8 (I1), U28.2 (OUT)
- new net Hall_51: U11.7 (I2), U36.2 (OUT)
- new net Hall_52: U11.6 (I3), U43.2 (OUT)
- new net Hall_53: U11.5 (I4), U51.2 (OUT)
- new net Hall_54: U11.4 (I5), U59.2 (OUT)
- new net Hall_55: U11.3 (I6), U67.2 (OUT)
- new net Hall_56: U11.2 (I7), U75.2 (OUT)
- new net Hall_57: U11.23 (I8), U21.2 (OUT)
- new net Hall_58: U11.22 (I9), U29.2 (OUT)
- new net Hall_59: U11.21 (I10), U37.2 (OUT)
- new net Hall_6: U53.2 (OUT), U7.4 (I5)
- new net Hall_60: U11.20 (I11), U44.2 (OUT)
- new net Hall_61: U11.19 (I12), U52.2 (OUT)
- new net Hall_62: U11.18 (I13), U60.2 (OUT)
- new net Hall_63: U11.17 (I14), U68.2 (OUT)
- new net Hall_64: U11.16 (I15), U76.2 (OUT)
- new net Hall_7: U61.2 (OUT), U7.3 (I6)
- new net Hall_8: U69.2 (OUT), U7.2 (I7)
- new net Hall_9: U15.2 (OUT), U7.23 (I8)
- new net S0: U10.10 (S0), U11.10 (S0), U7.10 (S0), U8.10 (S0)
- new net S1: U10.11 (S1), U11.11 (S1), U7.11 (S1), U8.11 (S1)
- new net S2: U10.14 (S2), U11.14 (S2), U7.14 (S2), U8.14 (S2)
- new net S3: U10.13 (S3), U11.13 (S3), U7.13 (S3), U8.13 (S3)
- new net SIG_1: U12.13 (B1), U7.1 (I/O)
- new net SIG_2: U12.12 (B2), U8.1 (I/O)
- new net SIG_3: U10.1 (I/O), U12.11 (B3)
- new net SIG_4: U11.1 (I/O), U12.10 (B4)
- no-connect marks 0 -> 1
Other:
- title: (none) -> SmartChessboard

Commit message: psc
Parts:
- removed U12: TXB0104D, Package_SO:SOIC-14_3.9x8.7mm_P1.27mm, symbol Logic_LevelTranslator:TXB0104D
- added C76, C77, C78, C79: 0.1uF, SparkFun-Capacitor:C_0402_1005Metric, symbol SparkFun-Capacitor:0.1uF_0402_6.3V_10%
- added Q2, Q3, Q4, Q5: BSS138, Package_TO_SOT_SMD:SOT-23, symbol Transistor_FET:BSS138
- added R13, R14, R15, R16, R17, R18, R19, R20, R29, R30, R39, R40: 10k, SparkFun-Resistor:R_0402_1005Metric, symbol SparkFun-Resistor:10k_0402
- renumbered C98 to C100, C99 to C101, C100 to C102, C101 to C103, C102 to C104, C103 to C105, C104 to C106, C105 to C107, C106 to C108, C107 to C109, C108 to C110, C109 to C111, C110 to C112, C111 to C113, C112 to C114, C113 to C115, C114 to C116, C115 to C117, C116 to C118, C117 to C119, C118 to C120, C119 to C121, C120 to C122, C121 to C123, C122 to C124, C123 to C125, C124 to C126, C125 to C127, C9 to C128, C126 to C129, C127 to C130, C128 to C131, C129 to C132, C130 to C133, C131 to C134, C132 to C135, C13 to C136, C133 to C137, C134 to C138, C135 to C139, C136 to C140, C137 to C141, C138 to C142, C139 to C143, C140 to C144, C141 to C145, C142 to C146, C143 to C147, C144 to C148, C145 to C149, C146 to C150, C147 to C151, C148 to C152, C149 to C153, C150 to C154, C151 to C155, C152 to C156, C153 to C157, C154 to C158, C155 to C159, C156 to C160, C157 to C161, C158 to C162, C159 to C163, C160 to C164, C161 to C165, C162 to C166, C163 to C167, C164 to C168, C165 to C169, C166 to C170, C167 to C171, C168 to C172, C169 to C173, C170 to C174, C171 to C175, C172 to C176, C173 to C177, C174 to C178, C175 to C179, C176 to C180, C177 to C181, C178 to C182, C179 to C183, C180 to C184, C181 to C185, C182 to C186, C183 to C187, C184 to C188, C185 to C189, C186 to C190, C187 to C191, C188 to C192, C189 to C193, C190 to C194, C191 to C195, C192 to C196, C193 to C197, C194 to C198, C195 to C199, C196 to C200, C197 to C201, C198 to C202, C199 to C203, C200 to C204, C201 to C205, C202 to C206, C203 to C207, C78 to C80, C79 to C81, C80 to C82, C81 to C83, C82 to C84, C83 to C85, C84 to C86, C85 to C87, C86 to C88, C87 to C89, C88 to C90, C89 to C91, C90 to C92, C91 to C93, C92 to C94, C93 to C95, C94 to C96, C95 to C97, C96 to C98, C97 to C99, R14 to R21, R15 to R22, R16 to R23, R17 to R24, R18 to R25, R19 to R26, R20 to R27, R21 to R28, R22 to R31, R23 to R32, R24 to R33, R25 to R34, R26 to R35, R27 to R36, R28 to R37, R29 to R38, R30 to R41, R31 to R42, R32 to R43, R33 to R44, R34 to R45, R35 to R46, R36 to R47, R37 to R48, R13 to R49, R38 to R50, R39 to R51, R40 to R52, R41 to R53, R42 to R54, R43 to R55, R44 to R56, R45 to R57, R46 to R58, R47 to R59, R48 to R60, R49 to R61, R50 to R62, R51 to R63, R52 to R64, R53 to R65, R54 to R66, R55 to R67, R56 to R68, R57 to R69, R58 to R70, R59 to R71, R60 to R72, R61 to R73, R62 to R74, R63 to R75, R64 to R76, R65 to R77, R66 to R78, R67 to R79, R68 to R80, R69 to R81, R70 to R82, R71 to R83, R72 to R84, R73 to R85, R74 to R86, R75 to R87, R76 to R88, U11 to U10, U14 to U11, U15 to U12, U16 to U13, U17 to U14, U18 to U15, U19 to U16, U20 to U17, U21 to U18, U22 to U19, U23 to U20, U24 to U21, U25 to U22, U26 to U23, U27 to U24, U28 to U25, U29 to U26, U30 to U27, U31 to U28, U32 to U29, U33 to U30, U34 to U31, U35 to U32, U36 to U33, U37 to U34, U9 to U35, U38 to U36, U39 to U37, U40 to U38, U41 to U39, U42 to U40, U43 to U41, U44 to U42, U45 to U43, U46 to U44, U47 to U45, U48 to U46, U49 to U47, U50 to U48, U51 to U49, U52 to U50, U53 to U51, U54 to U52, U55 to U53, U56 to U54, U57 to U55, U58 to U56, U59 to U57, U60 to U58, U61 to U59, U62 to U60, U63 to U61, U64 to U62, U65 to U63, U66 to U64, U67 to U65, U68 to U66, U69 to U67, U70 to U68, U71 to U69, U72 to U70, U73 to U71, U74 to U72, U75 to U73, U76 to U74, U10 to U9
Connections:
- net 3.3V: now also Q2.1 (G), Q3.1 (G), Q4.1 (G), Q5.1 (G), R17.1, R19.1, R29.1, R39.1
- net 5V: now also C76.1, C77.1, C78.1, C79.1, R18.1, R20.1, R30.1, R40.1
- net GND: now also C76.2, C77.2, C78.2, C79.2, R13.1, R13.2, R14.1, R14.2, R15.1, R15.2, R16.1, R16.2
- net SIG_1: now also Q2.3 (D), R18.2
- net SIG_2: now also Q3.3 (D), R20.2
- net SIG_3: now also Q4.3 (D), R30.2
- net SIG_4: now also Q5.3 (D), R40.2
- new net LV_SIG_1: Q2.2 (S), R17.2
- new net LV_SIG_2: Q3.2 (S), R19.2
- new net LV_SIG_3: Q4.2 (S), R29.2
- new net LV_SIG_4: Q5.2 (S), R39.2
- no-connect marks 1 -> 0
Other:
- note added: "Bidirectional Logic Level Converter"
- note added: "Multiplexer"
- moved on the sheet: U10, U7, U8, U9

Commit message: added pwr management pcb
Parts:
- added JP3: ~, SparkFun-Jumper:Jumper_2_NC_Trace, symbol SparkFun-Jumper:SolderJumper_2_Bridged
Connections:
- net 5V: now also JP3.1 (A), JP3.2 (B)
- net Hall_1: no longer C104.1, C105.1, C106.1, C107.1, C108.1, C109.1, C110.1, C111.1, C120.1, C121.1, C122.1, C123.1, C124.1, C125.1, C126.1, C127.1, C136.1, C137.1, C138.1, C139.1, C140.1, C141.1, C142.1, C143.1, C152.1, C153.1, C154.1, C155.1, C156.1, C157.1, C158.1, C159.1, C168.1, C169.1, C170.1, C171.1, C172.1, C173.1, C174.1, C175.1, C184.1, C185.1, C186.1, C187.1, C188.1, C189.1, C190.1, C191.1, C200.1, C201.1, C202.1, C203.1, C204.1, C205.1, C206.1, C207.1, C89.1, C90.1, C91.1, C92.1, C93.1, C94.1, C95.1, R22.1, R23.1, R24.1, R25.1, R26.1, R27.1, R28.1, R31.1, R32.1, R33.1, R34.1, R35.1, R36.1, R37.1, R38.1, R41.1, R42.1, R43.1, R44.1, R45.1, R46.1, R47.1, R48.1, R49.1, R50.1, R51.1, R52.1, R53.1, R54.1, R55.1, R56.1, R57.1, R58.1, R59.1, R60.1, R61.1, R62.1, R63.1, R64.1, R65.1, R66.1, R67.1, R68.1, R69.1, R70.1, R71.1, R72.1, R73.1, R74.1, R75.1, R76.1, R77.1, R78.1, R79.1, R80.1, R81.1, R82.1, R83.1, R84.1, R85.1, R86.1, R87.1, R88.1
- net Hall_10: now also C105.1, R32.1
- net Hall_11: now also C121.1, R42.1
- net Hall_12: now also C137.1, R50.1
- net Hall_13: now also C153.1, R58.1
- net Hall_14: now also C169.1, R66.1
- net Hall_15: now also C185.1, R74.1
- net Hall_16: now also C201.1, R82.1
- net Hall_17: now also C90.1, R23.1
- net Hall_18: now also C106.1, R33.1
- net Hall_19: now also C122.1, R43.1
- net Hall_2: now also C104.1, R31.1
- net Hall_20: now also C138.1, R51.1
- net Hall_21: now also C154.1, R59.1
- net Hall_22: now also C170.1, R67.1
- net Hall_23: now also C186.1, R75.1
- net Hall_24: now also C202.1, R83.1
- net Hall_25: now also C91.1, R24.1
- net Hall_26: now also C107.1, R34.1
- net Hall_27: now also C123.1, R44.1
- net Hall_28: now also C139.1, R52.1
- net Hall_29: now also C155.1, R60.1
- net Hall_3: now also C120.1, R41.1
- net Hall_30: now also C171.1, R68.1
- net Hall_31: now also C187.1, R76.1
- net Hall_32: now also C203.1, R84.1
- net Hall_33: now also C92.1, R25.1
- net Hall_34: now also C108.1, R35.1
- net Hall_35: now also C124.1, R45.1
- net Hall_36: now also C140.1, R53.1
- net Hall_37: now also C156.1, R61.1
- net Hall_38: now also C172.1, R69.1
- net Hall_39: now also C188.1, R77.1
- net Hall_4: now also C136.1, R49.1
- net Hall_40: now also C204.1, R85.1
- net Hall_41: now also C93.1, R26.1
- net Hall_42: now also C109.1, R36.1
- net Hall_43: now also C125.1, R46.1
- net Hall_44: now also C141.1, R54.1
- net Hall_45: now also C157.1, R62.1
- net Hall_46: now also C173.1, R70.1
- net Hall_47: now also C189.1, R78.1
- net Hall_48: now also C205.1, R86.1
- net Hall_49: now also C94.1, R27.1
- net Hall_5: now also C152.1, R57.1
- net Hall_50: now also C110.1, R37.1
- net Hall_51: now also C126.1, R47.1
- net Hall_52: now also C142.1, R55.1
- net Hall_53: now also C158.1, R63.1
- net Hall_54: now also C174.1, R71.1
- net Hall_55: now also C190.1, R79.1
- net Hall_56: now also C206.1, R87.1
- net Hall_57: now also C95.1, R28.1
- net Hall_58: now also C111.1, R38.1
- net Hall_59: now also C127.1, R48.1
- net Hall_6: now also C168.1, R65.1
- net Hall_60: now also C143.1, R56.1
- net Hall_61: now also C159.1, R64.1
- net Hall_62: now also C175.1, R72.1
- net Hall_63: now also C191.1, R80.1
- net Hall_64: now also C207.1, R88.1
- net Hall_7: now also C184.1, R73.1
- net Hall_8: now also C200.1, R81.1
- net Hall_9: now also C89.1, R22.1

Commit message: pcb finished
Connections:
- net GND: no longer R13.2, R14.2, R15.2, R16.2, U10.15 (~{EN}), U7.15 (~{EN}), U8.15 (~{EN}), U9.15 (~{EN})
- new net: R13.2, U7.15 (~{EN})
- new net: R14.2, U8.15 (~{EN})
- new net: R16.2, U10.15 (~{EN})
- new net: R15.2, U9.15 (~{EN})
